File: kicad/mpu_power_clock.kicad_sch (KiCad schematic)
At the start: 50 parts, among them SW201 Omron B3F-1052, SW202 SW_DIP_x04, U201 NCP380, U202 STM32MP135FAEx, Y201 24 MHz

Commit message: board as built
Parts:
- C224, C228: JLCPCB C1523 -> C12530
Changed lines of the file:
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@@
 			)
 		)
-		(property "JLCPCB" "C1523"
+		(property "JLCPCB" " C12530"
 			(at 295.91 146.05 0)
 			(effects
@@
 			)
 		)
-		(property "JLCPCB" "C1523"
+		(property "JLCPCB" " C12530"
 			(at 287.02 146.05 0)
 			(effects
